Commit message: feat: le drone cartographie par vision, le robot planifie et suit en MPC
Le robot ne lit plus aucun fichier et le drone ne reçoit aucune dimension :
la carte est entièrement redécouverte depuis une image caméra nadir, publiée
en nav_msgs/OccupancyGrid latchée, puis replanifiée en A* par le robot.

Vision (maze_vision.py)
  - Segmentation HSV des murs ; la pastille d'arrivée, de la même couleur, est
    séparée par sa forme et non par sa teinte.
  - rows, cols et la taille de cellule sont inférés conjointement des lignes de
    grille sous contrainte de cellules carrées — une erreur de facteur 2 sur un
    seul axe est trahie par le rapport des pas.
  - La parallaxe des murs est résolue à partir des deux bords de leur bande, ce
    qui ramène chaque ligne au plan du sol sans connaître leur épaisseur. Sans
    cela le labyrinthe est reconstruit systématiquement trop petit.
  - Vote sur plusieurs images : manquer un mur autorise un chemin qui traverse
    une cloison, en inventer un ne coûte qu'un détour.
  - Un échec lève une exception plutôt que de rendre une grille douteuse.

Commande (mpc_controller.py)
  - MPC CasADi/IPOPT, horizon 1,8 s, modèle unicycle intégré au point milieu.
  - Les murs sont des pénalités douces : une contrainte dure devient infaisable
    dès que le robot dérive dans la marge, et le solveur renvoie une erreur au
    moment où l'on en a le plus besoin.
  - Le terme (v·sin Δθ)² est la version continue et anticipative du cos(err)^8.
  - Réamorçage à chaud conservé même après un échec, sans quoi un échec isolé
    dégénère en cascade ; invalidé explicitement quand le problème change.
  - Plafond de temps de résolution : le nœud est mono-thread, un solveur qui
    s'éternise fige aussi la lecture de l'odométrie.

Drone (drone_mapper_node.py)
  - Cadrage autonome : le drone décolle dans un coin du labyrinthe et ajuste
    seul position et altitude jusqu'à tout cadrer, quelle que soit la taille.
  - Correction de l'assiette du drone dans la projection : deux degrés de
    tangage résiduel translataient la carte de 10 cm.
  - Nouvel état RETURN_TO_ROBOT : READY n'est publié qu'une fois le drone revenu
    à 1 m au-dessus du robot et stabilisé sur son marqueur, sinon le suivi
    démarrerait en rattrapage.

Correctif de modélisation (robot_core.xacro)
  - Le visuel du lien IMU dépassait de 4 mm au-dessus du plan du marqueur ArUco,
    pile en son centre, et corrompait la lecture des bits. Logé au centre du
    châssis, le taux de détection passe de 40 % à 91 %.

Validation (maze_map_validator.py, validate_map:=true)
  Grilles 4x4, 5x5 et 6x6 : 64/64, 100/100 et 144/144 arêtes correctes, chemin
  A* identique au réel, cellule à 0,4-1,0 mm près, origine à 2-3 mm.
  Limite connue : la dérive odométrique atteint ~6,6 cm à l'arrivée, au-dessus
  des 5 cm visés. Elle est longitudinale et vient du glissement au freinage, la
  roue folle étant quasi sans frottement ; la corriger demanderait une fusion
  odométrie/IMU, hors périmètre ici.

File: description/robot_core.xacro (robot description, xacro)
@@ -142,5 +142,14 @@
     <parent link="chassis_link"/>
     <child link="imu_link"/>
-    <origin xyz="0 0 ${chassis_height/2.0}" rpy="0 0 0"/>
+    <!--
+      L'IMU est logée AU CENTRE du châssis, pas sur sa face supérieure.
+      Posée sur le dessus, sa boîte visuelle de 2 cm dépassait de 4 mm au-dessus
+      du plan du marqueur ArUco et se retrouvait pile en son centre : le drone
+      voyait alors un carré rouge au milieu du motif, les bits étaient corrompus
+      et le marqueur n'était reconnu qu'une image sur deux. Au centre, elle est
+      entièrement enfermée dans le châssis — et c'est de toute façon la place
+      naturelle d'une centrale inertielle.
+    -->
+    <origin xyz="0 0 0" rpy="0 0 0"/>
   </joint>
   <!-- ============================ ARUCO MARKER (top) ============================ -->
